File: doc/schematics/module/eavesdrum.kicad_pcb (KiCad board)
At the start: 2 copper layers, 100 x 100 mm, 100 parts, among them J1 DC37_Pins_MountingHoles, J2 Conn_02x25_Odd_Even, J3 Conn_01x03, M4_1 MountingHole_4.3mm_M4, M4_2 MountingHole_4.3mm_M4, M4_3 MountingHole_4.3mm_M4, M4_4 MountingHole_4.3mm_M4, SW1 SW_Push, SW2 SW_Push, SW3 SW_Push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

Commit message: adjust module schematics
Routing:
- net /addr1_1: track 107.5 -> 104.4 mm, vias 3 -> 5
- net /in2_14: track 72.1 -> 73.5 mm
- net /addr2_0: track 70.6 -> 71.3 mm
- net GND: vias 237 -> 239

Commit message: fix pcba issues
Parts:
- moved R3 2.50 mm to (85.0, 50.0)
- moved R6 2.45 mm to (97.0, 50.0)
- moved D3 1.30 mm to (123.8, 48.2)
- moved D4 1.28 mm to (116.0, 48.2)
- moved JP1 0.88 mm to (118.7, 120.5)
- moved JP2 0.84 mm to (128.5, 120.5)
- moved JP3 0.84 mm to (138.5, 120.5)
- moved JP5 0.84 mm to (158.0, 120.5)
- moved JP4 0.80 mm to (148.2, 120.5)
- moved R10 0.72 mm to (116.0, 43.8)
- moved R9 0.72 mm to (124.0, 43.8)
Routing:
- net /in2_7: track 208.4 -> 55.9 mm, vias 7 -> 3
- net /in2_5: track 190.0 -> 53.2 mm, vias 6 -> 1
- net /in2_9: track 68.6 -> 134.5 mm, vias 5 -> 8
- net /in2_8: track 69.0 -> 124.7 mm, vias 4 -> 8
- net /in2_12: track 83.2 -> 53.3 mm, vias 5 -> 1
- net Net-(D2.14-COM): track 76.8 -> 102.5 mm, vias 4 -> 6
- net /in2_15: track 65.1 -> 90.4 mm, vias 1 -> 3
- net Net-(D2.1-COM): track 70.2 -> 45.4 mm, vias 5 -> 3
- net GND: track 606.0 -> 581.3 mm, vias 239 -> 238
- net +3.3V: track 335.5 -> 313.6 mm, vias 5 -> 9
- net Net-(D2.2-COM): track 72.5 -> 53.1 mm, vias 4 -> 3
- net Net-(D2.6-COM): track 89.6 -> 70.6 mm, vias 9 -> 2
- net Net-(D2.12-COM): track 100.1 -> 81.7 mm, vias 6 -> 3
- net /gpio20: track 100.2 -> 81.7 mm
- net /nEna1: track 89.2 -> 106.6 mm
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