File: doc/schematics/connector/eavesdrum_connector.kicad_pcb (KiCad board)
At the start: 2 copper layers, 100 x 100 mm, 20 parts, among them J1 AudioJack3_Dual_Ground_Switch, J10 AudioJack3_Dual_Ground_Switch, J11 AudioJack3_Dual_Ground_Switch, J12 SUB-D 44 HD, J13 Conn_01x03_Pin, J14 Conn_01x07_Pin, J2 AudioJack3_Dual_Ground_Switch, J3 AudioJack3_Dual_Ground_Switch, J4 AudioJack3_Dual_Ground_Switch, J5 AudioJack3_Dual_Ground_Switch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

Commit message: update schematics
Parts:
- added JP7: Jumper_3_Open, Connector_PinHeader_2.54mm:PinHeader_1x03_P2.54mm_Vertical, F.Cu at (168.2, 97.1)
- added JP8: Jumper_3_Open, Connector_PinHeader_2.54mm:PinHeader_1x03_P2.54mm_Vertical, F.Cu at (168.2, 106.9)
Connections:
- J11 pad 2(4): unconnected-(J11B-R2-Pad2(4)) -> Net-(J11B-R2)
- J11 pad 4: unconnected-(J11A-R1-Pad4) -> Net-(J11A-R1)
Routing:
- net +3.3V: track 60.9 -> 107.0 mm, vias 0 -> 1
- net /in2_1: track 125.6 -> 90.2 mm, vias 4 -> 2
- net /in2_10: track 61.0 -> 96.3 mm
- net /in2_12: track 65.4 -> 97.3 mm, vias 1 -> 2
- net GND: track 340.8 -> 372.6 mm, vias 538 -> 503
- net +5V: track 79.3 -> 106.0 mm, vias 1 -> 2
- net Net-(J11A-R1): track 0.00 -> 22.9 mm
- net Net-(J11B-R2): track 0.00 -> 17.4 mm
- net /in1_11: track 150.5 -> 134.4 mm, vias 1 -> 2
- net /in1_2: track 66.3 -> 81.9 mm, vias 1 -> 2
- net /in2_6: track 104.4 -> 90.0 mm, vias 3 -> 6
- net /in1_8: track 90.8 -> 104.3 mm
- net gpio16: track 82.3 -> 69.8 mm
- net /in2_14: track 109.8 -> 100.8 mm, vias 2 -> 1
- net /in2_8: track 96.7 -> 89.0 mm, vias 1 -> 2
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Other:
- board text added: "Pedal1 (Hi-Hat) Pedal2"
- board text removed: "Hi-Hat Pedal (Resistive) Hi-Hat Pedal (Optical)"
