File: doc/schematics/connector/eavesdrum_connector.kicad_sch (KiCad schematic)
At the start: 20 parts, among them J1 AudioJack3_Dual_Ground_Switch, J10 AudioJack3_Dual_Ground_Switch, J11 AudioJack3_Dual_Ground_Switch, J12 SUB-D 44 HD, J13 Conn_01x03_Pin, J14 Conn_01x07_Pin, J2 AudioJack3_Dual_Ground_Switch, J3 AudioJack3_Dual_Ground_Switch, J4 AudioJack3_Dual_Ground_Switch, J5 AudioJack3_Dual_Ground_Switch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

Commit message: update schematics
Parts:
- added JP7, JP8: Jumper_3_Open, Connector_PinHeader_2.54mm:PinHeader_1x03_P2.54mm_Vertical, symbol Jumper:Jumper_3_Open
Connections:
- net +3.3V: now also JP7.1 (A), JP8.1 (A)
- net +5V: now also JP7.3 (B), JP8.3 (B)
- net at J11.4 (R1): now also JP8.2 (C)
- net at J11.2(4) (R2): now also JP7.2 (C)
- no-connect marks 70 -> 68
